File: qris_iot.kicad_sch (KiCad schematic)
At the start: 0 parts

Commit message: anjir
Other:
- removed sheet Uarts
- added sheet batere (batere.kicad_sch)
- added sheet gnss_quectell (gnss_quectel.kicad_sch)
- added sheet servo (servo.kicad_sch)
Changed lines of the file:
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@@
 	(paper "A4")
 	(sheet
-		(at 106.68 34.29)
-		(size 27.94 12.7)
+		(at 106.68 33.02)
+		(size 30.48 13.97)
 		(fields_autoplaced yes)
 		(stroke
@@
 		)
 		(property "Sheetname" "Power Supply"
-			(at 106.68 33.5784 0)
+			(at 106.68 32.3084 0)
 			(effects
 				(font
@@
 	)
 	(sheet
-		(at 139.7 34.29)
-		(size 22.86 12.7)
+		(at 139.7 33.02)
+		(size 25.4 13.97)
 		(fields_autoplaced yes)
 		(stroke
@@
 		)
 		(property "Sheetname" "Memory"
-			(at 139.7 33.5784 0)
+			(at 139.7 32.3084 0)
 			(effects
 				(font
@@
 	)
 	(sheet
-		(at 138.43 54.61)
-		(size 21.59 8.89)
+		(at 176.53 53.34)
+		(size 27.94 17.78)
+		(fields_autoplaced yes)
+		(stroke
+			(width 0.1524)
+			(type solid)
+		)
+		(fill
+			(color 0 0 0 0.0000)
+		)
+		(property "Sheetname" "batere"
+			(at 176.53 52.6284 0)
+			(effects
+				(font
+					(size 1.27 1.27)
+				)
+				(justify left bottom)
+			)
+		)
+		(property "Sheetfile" "batere.kicad_sch"
+			(at 176.53 71.7046 0)
+			(effects
+				(font
+					(size 1.27 1.27)
+				)
+				(justify left top)
+			)
+		)
+		(instances
+			(project "qris_iot"
+				(path "/7e5ed2de-adc7-481a-a10e-7326381f5ab2"
+					(page "10")
+				)
+			)
+		)
+	)
+	(sheet
+		(at 138.43 53.34)
+		(size 22.86 10.16)
 		(fields_autoplaced yes)
 		(stroke
@@
 		)
 		(property "Sheetname" "JTAG"
-			(at 138.43 53.8984 0)
+			(at 138.43 52.6284 0)
 			(effects
 				(font
@@
 	)
 	(sheet
-		(at 138.43 93.98)
-		(size 24.13 13.97)
+		(at 199.39 86.36)
+		(size 33.02 17.78)
+		(fields_autoplaced yes)
+		(stroke
+			(width 0.1524)
+			(type solid)
+		)
+		(fill
+			(color 0 0 0 0.0000)
+		)
+		(property "Sheetname" "servo"
+			(at 199.39 85.6484 0)
+			(effects
+				(font
+					(size 1.27 1.27)
+				)
+				(justify left bottom)
+			)
+		)
+		(property "Sheetfile" "servo.kicad_sch"
+			(at 199.39 104.7246 0)
+			(effects
+				(font
+					(size 1.27 1.27)
+				)
+				(justify left top)
+			)
+		)
+		(instances
+			(project "qris_iot"
+				(path "/7e5ed2de-adc7-481a-a10e-7326381f5ab2"
+					(page "9")
+				)
+			)
+		)
+	)
+	(sheet
+		(at 153.67 88.9)
+		(size 24.13 24.13)
 		(fields_autoplaced yes)
 		(stroke
@@
 		)
 		(property "Sheetname" "quectell"
-			(at 138.43 93.2684 0)
+			(at 153.67 88.1884 0)
 			(effects
 				(font
@@
 		)
 		(property "Sheetfile" "quectell.kicad_sch"
-			(at 138.43 108.5346 0)
+			(at 153.67 113.6146 0)
 			(effects
 				(font
@@
 	)
 	(sheet
-		(at 138.43 71.12)
-		(size 25.4 12.7)
+		(at 125.73 72.39)
+		(size 21.59 8.89)
 		(fields_autoplaced yes)
 		(stroke
@@
 		)
 		(property "Sheetname" "LCD"
-			(at 138.43 70.4084 0)
+			(at 125.73 71.6784 0)
 			(effects
 				(font
@@
 		)
 		(property "Sheetfile" "LCD.kicad_sch"
-			(at 138.43 84.4046 0)
+			(at 125.73 81.8646 0)
 			(effects
 				(font
@@
 	)
 	(sheet
-		(at 106.68 54.61)
-		(size 27.94 8.89)
+		(at 114.3 93.98)
+		(size 30.48 12.7)
+		(fields_autoplaced yes)
+		(stroke
+			(width 0.1524)
+			(type solid)
+		)
+		(fill
+			(color 0 0 0 0.0000)
+		)
+		(property "Sheetname" "gnss_quectell"
+			(at 114.3 93.2684 0)
+			(effects
+				(font
+					(size 1.27 1.27)
+				)
+				(justify left bottom)
+			)
+		)
+		(property "Sheetfile" "gnss_quectel.kicad_sch"
+			(at 114.3 107.2646 0)
+			(effects
+				(font
+					(size 1.27 1.27)
+				)
+				(justify left top)
+			)
+		)
+		(instances
+			(project "qris_iot"
+				(path "/7e5ed2de-adc7-481a-a10e-7326381f5ab2"
+					(page "9")
+				)
+			)
+		)
+	)
+	(sheet
+		(at 106.68 53.34)
+		(size 30.48 10.16)
 		(fields_autoplaced yes)
 		(stroke
@@
 		)
 		(property "Sheetname" "MIMXRT1010"
-			(at 106.68 53.8984 0)
+			(at 106.68 52.6284 0)
 			(effects
 				(font
@@
 				)
 			)
-		)
-	)
-	(sheet
-		(at 106.68 69.85)
-		(size 25.4 15.24)
-		(fields_autoplaced yes)
-		(stroke
-			(width 0.1524)
-			(type solid)
-		)
-		(fill
-			(color 0 0 0 0.0000)
-		)
-		(property "Sheetname" "Uarts"
-			(at 106.68 69.1384 0)
-			(effects
-				(font
-					(size 1.27 1.27)
-				)
-				(justify left bottom)
-			)
-		)
-		(property "Sheetfile" "uarts.kicad_sch"
-			(at 106.68 85.6746 0)
-			(effects
-				(font
-					(size 1.27 1.27)
-				)
-				(justify left top)
-			)
-		)
-		(instances
-			(project "qris_iot"
-				(path "/7e5ed2de-adc7-481a-a10e-7326381f5ab2"
-					(page "7")
-				)
-			)

Commit message: yara me kya karun
Other:
- added sheet keypad (keypad.kicad_sch)
- added sheet printer (printer.kicad_sch)
Changed lines of the file:
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@@
+	)
+	(sheet
+		(at 218.44 36.83)
+		(size 22.86 17.78)
+		(fields_autoplaced yes)
+		(stroke
+			(width 0.1524)
+			(type solid)
+		)
+		(fill
+			(color 0 0 0 0.0000)
+		)
+		(property "Sheetname" "printer"
+			(at 218.44 36.1184 0)
+			(effects
+				(font
+					(size 1.27 1.27)
+				)
+				(justify left bottom)
+			)
+		)
+		(property "Sheetfile" "printer.kicad_sch"
+			(at 218.44 55.1946 0)
+			(effects
+				(font
+					(size 1.27 1.27)
+				)
+				(justify left top)
+			)
+		)
+		(instances
+			(project "qris_iot"
+				(path "/7e5ed2de-adc7-481a-a10e-7326381f5ab2"
+					(page "11")
+				)
+			)
+		)
 	)
 	(sheet
@@
 				)
 			)
+		)
+	)
+	(sheet
+		(at 184.15 120.65)
+		(size 27.94 15.24)
+		(fields_autoplaced yes)
+		(stroke
+			(width 0.1524)
+			(type solid)
+		)
+		(fill
+			(color 0 0 0 0.0000)
+		)
+		(property "Sheetname" "keypad"
+			(at 184.15 119.9384 0)
+			(effects
+				(font
+					(size 1.27 1.27)
+				)
+				(justify left bottom)
+			)
+		)
+		(property "Sheetfile" "keypad.kicad_sch"
+			(at 184.15 136.4746 0)
+			(effects
+				(font
+					(size 1.27 1.27)
+				)
+				(justify left top)
+			)
+		)
+		(instances
+			(project "qris_iot"
+				(path "/7e5ed2de-adc7-481a-a10e-7326381f5ab2"
+					(page "12")
+				)
+			)

Commit message: sebelum pemeriksaan terkahir
Other:
- removed sheet batere
- added sheet PMIC (PMIC.kicad_sch)
- added sheet battery (battery.kicad_sch)
Changed lines of the file:
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@@
 	)
 	(sheet
-		(at 176.53 53.34)
-		(size 27.94 17.78)
+		(at 177.8 55.88)
+		(size 25.4 21.59)
 		(fields_autoplaced yes)
 		(stroke
@@
 			(color 0 0 0 0.0000)
 		)
-		(property "Sheetname" "batere"
-			(at 176.53 52.6284 0)
+		(property "Sheetname" "battery"
+			(at 177.8 55.1684 0)
 			(effects
 				(font
@@
 			)
 		)
-		(property "Sheetfile" "batere.kicad_sch"
-			(at 176.53 71.7046 0)
+		(property "Sheetfile" "battery.kicad_sch"
+			(at 177.8 78.0546 0)
 			(effects
 				(font
@@
 			(project "qris_iot"
 				(path "/7e5ed2de-adc7-481a-a10e-7326381f5ab2"
-					(page "10")
+					(page "13")
 				)
 			)
@@
 				)
 			)
+		)
+	)
+	(sheet
+		(at 129.54 129.54)
+		(size 34.29 19.05)
+		(fields_autoplaced yes)
+		(stroke
+			(width 0.1524)
+			(type solid)
+		)
+		(fill
+			(color 0 0 0 0.0000)
+		)
+		(property "Sheetname" "PMIC"
+			(at 129.54 128.8284 0)
+			(effects
+				(font
+					(size 1.27 1.27)
+				)
+				(justify left bottom)
+			)
+		)
+		(property "Sheetfile" "PMIC.kicad_sch"
+			(at 129.54 149.1746 0)
+			(effects
+				(font
+					(size 1.27 1.27)
+				)
+				(justify left top)
+			)
+		)
+		(instances
+			(project "qris_iot"
+				(path "/7e5ed2de-adc7-481a-a10e-7326381f5ab2"
+					(page "13")
+				)
+			)
