File: printer.kicad_sch (KiCad schematic)
At the start: 1 part, among them J6 Conn_01x04_Pin

Commit message: da
Changed lines of the file:
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@@
 		)
 	)
-	(label "LPUART4_TXD_ALT0"
+	(global_label "LPUART4_TXD_ALT0"
+		(shape input)
 		(at 124.46 77.47 180)
 		(fields_autoplaced yes)
@@
 				(size 1.27 1.27)
 			)
-			(justify right bottom)
+			(justify right)
+		)
+		(property "Intersheetrefs" "${INTERSHEET_REFS}"
+			(at 103.6344 77.47 0)
+			(effects
+				(font
+					(size 1.27 1.27)
+				)
+				(justify right)
+				(hide yes)
+			)
 		)
 	)
-	(label "LPUART4_RXD_ALT0"
+	(global_label "LPUART4_RXD_ALT0"
+		(shape input)
 		(at 124.46 74.93 180)
 		(fields_autoplaced yes)
@@
 				(size 1.27 1.27)
 			)
-			(justify right bottom)
+			(justify right)
+		)
+		(property "Intersheetrefs" "${INTERSHEET_REFS}"
+			(at 103.332 74.93 0)
+			(effects
+				(font
+					(size 1.27 1.27)
+				)
+				(justify right)
+				(hide yes)
+			)
 		)
 	)
-	(label "3V3_UART4"
+	(global_label "3V3_UART4"
+		(shape input)
 		(at 130.81 59.69 0)
 		(fields_autoplaced yes)
@@
 				(size 1.27 1.27)
 			)
-			(justify left bottom)
+			(justify left)
+		)
+		(property "Intersheetrefs" "${INTERSHEET_REFS}"
+			(at 144.1366 59.69 0)
+			(effects
+				(font
+					(size 1.27 1.27)
+				)
+				(justify left)
+				(hide yes)
+			)
 		)
 	)
